File: Adapter-IO4-Molex156.brd (EAGLE design)
At the start: 30.9 x 31.9 mm, 3 parts

Commit message: 1.1
Parts:
- moved U$1 27.8 mm to (4.67, 45.6)
- moved J4 20.3 mm to (25.2, 44.3)
- moved X1 10.0 mm to (25.2, 7.46)
Routing:
- net VCC: track 14.3 -> 34.3 mm
- net GND: track 17.6 -> 36.8 mm
- net IO3: track 13.5 -> 31.2 mm, vias 0 -> 2
- net IO2: track 10.8 -> 28.5 mm
- net IO1: track 14.4 -> 32.2 mm
- net IO4: track 11.8 -> 29.6 mm
- added copper zone on layer 16, net GND
- removed copper zone on layer 16, net N$1
Other:
- board size 30.9 x 31.9 mm -> 50 x 50 mm
- board text added: "0.156 Pitch"
- board text added: "0.156 pitch"
- board text added: "2014.02"
- board text added: "IO4 Adapter"
- board text added: "IO4-Breakout"
- board text added: "v1.1"
- board text removed: "2012.08"
- board text removed: "Breakout"
- board text removed: "IOShield"
- board text removed: "IOShield Adapter"
- board text removed: "Lines"
- board text removed: "SPCoast"
- board text removed: "v1.0"

Commit message: added values for connectors
Parts:
- J4: value (none) -> RJ12/6
- X1: value (none) -> 0.156
Changed lines of the file:
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@@
 <elements>
 <element name="U$1" library="SPCoast" package="OSHW-LOGO-M" value="DOC-OSHW-LOGO-M" x="4.666" y="45.56"/>
-<element name="J4" library="SPCoast" package="RJ25-PANEL" value="" x="25.24" y="44.29" smashed="yes" rot="R180">
+<element name="J4" library="SPCoast" package="RJ25-PANEL" value="RJ12/6" x="25.24" y="44.29" smashed="yes" rot="R180">
 <attribute name="NAME" x="23.335" y="46.83" size="1.778" layer="25"/>
 <attribute name="VALUE" x="32.225" y="51.91" size="1.778" layer="27" rot="R180"/>
@@
 <attribute name="OPL" value="none" x="25.24" y="44.29" size="1.778" layer="27" rot="R180" display="off"/>
 </element>
-<element name="X1" library="SPCoast" package="KK-156-6" value="" x="25.24" y="7.46">
+<element name="X1" library="SPCoast" package="KK-156-6" value="0.156" x="25.24" y="7.46">
 <attribute name="MF" value="" x="25.24" y="7.46" size="1.778" layer="27" display="off"/>
 <attribute name="MPN" value="" x="25.24" y="7.46" size="1.778" layer="27" display="off"/>

Commit message: normalized values
Parts:
- U$1: value DOC-OSHW-LOGO-M -> OSHW
Changed lines of the file:
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@@
 </autorouter>
 <elements>
-<element name="U$1" library="SPCoast" package="OSHW-LOGO-M" value="DOC-OSHW-LOGO-M" x="4.666" y="45.56"/>
+<element name="U$1" library="SPCoast" package="OSHW-LOGO-M" value="OSHW" x="4.666" y="45.56"/>
 <element name="J4" library="SPCoast" package="RJ25-PANEL" value="RJ12/6" x="25.24" y="44.29" smashed="yes" rot="R180">
 <attribute name="NAME" x="23.335" y="46.83" size="1.778" layer="25"/>
