File: Adapter-IO4-Molex156.sch (EAGLE design)
At the start: 3 parts

Commit message: 1.1
Other:
- note added: "v1.1"
- note removed: "v1.0"
Changed lines of the file:
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@@
 <part name="J4" library="SPCoast" deviceset="CONNECTOR-RJ25" device="-6P6C"/>
 <part name="X1" library="SPCoast" deviceset="KK-156-6" device=""/>
+<part name="SUPPLY1" library="SparkFun-Aesthetics" deviceset="VCC" device=""/>
+<part name="GND1" library="SparkFun-Aesthetics" deviceset="GND" device=""/>
 </parts>
 <sheets>
@@
 <text x="152.4" y="27.94" size="3.81" layer="104">IOShield Breakout</text>
 <text x="208.28" y="27.94" size="3.81" layer="104">RJ11 adapter</text>
-<text x="236.22" y="7.62" size="3.81" layer="104">v1.0</text>
+<text x="236.22" y="7.62" size="3.81" layer="104">v1.1</text>
 </plain>
 <instances>
@@
 <instance part="X1" gate="-5" x="119.38" y="99.06" rot="R180"/>
 <instance part="X1" gate="-6" x="119.38" y="101.6" rot="R180"/>
+<instance part="SUPPLY1" gate="1" x="124.46" y="101.6"/>
+<instance part="GND1" gate="1" x="124.46" y="86.36"/>
 </instances>
 <busses>
@@
 <net name="VCC" class="0">
 <segment>
-<wire x1="129.54" y1="101.6" x2="121.92" y2="101.6" width="0.1524" layer="91"/>
+<wire x1="129.54" y1="101.6" x2="124.46" y2="101.6" width="0.1524" layer="91"/>
 <pinref part="J4" gate="J" pin="1"/>
 <pinref part="X1" gate="-6" pin="S"/>
+<pinref part="SUPPLY1" gate="1" pin="VCC"/>
+<wire x1="124.46" y1="101.6" x2="121.92" y2="101.6" width="0.1524" layer="91"/>
+<junction x="124.46" y="101.6"/>
 </segment>
 </net>
@@
 <net name="GND" class="0">
 <segment>
-<wire x1="129.54" y1="88.9" x2="121.92" y2="88.9" width="0.1524" layer="91"/>
+<wire x1="129.54" y1="88.9" x2="124.46" y2="88.9" width="0.1524" layer="91"/>
 <pinref part="J4" gate="J" pin="6"/>
 <pinref part="X1" gate="-1" pin="S"/>
+<pinref part="GND1" gate="1" pin="GND"/>
+<wire x1="124.46" y1="88.9" x2="121.92" y2="88.9" width="0.1524" layer="91"/>
+<junction x="124.46" y="88.9"/>
 </segment>
 </net>

Commit message: added values for connectors
Parts:
- J4: value (none) -> RJ12/6
- X1: value (none) -> 0.156
Changed lines of the file:
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@@
 <part name="FRAME1" library="SparkFun" deviceset="FRAME-LETTER" device=""/>
 <part name="U$1" library="SPCoast" deviceset="DOC-OSHW-LOGO-" device="M"/>
-<part name="J4" library="SPCoast" deviceset="CONNECTOR-RJ25" device="-6P6C"/>
-<part name="X1" library="SPCoast" deviceset="KK-156-6" device=""/>
+<part name="J4" library="SPCoast" deviceset="CONNECTOR-RJ25" device="-6P6C" value="RJ12/6"/>
+<part name="X1" library="SPCoast" deviceset="KK-156-6" device="" value="0.156"/>
 <part name="SUPPLY1" library="SparkFun-Aesthetics" deviceset="VCC" device=""/>
 <part name="GND1" library="SparkFun-Aesthetics" deviceset="GND" device=""/>

Commit message: normalized values
Parts:
- U$1: value DOC-OSHW-LOGO-M -> OSHW
Changed lines of the file:
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@@
 <parts>
 <part name="FRAME1" library="SparkFun" deviceset="FRAME-LETTER" device=""/>
-<part name="U$1" library="SPCoast" deviceset="DOC-OSHW-LOGO-" device="M"/>
+<part name="U$1" library="SPCoast" deviceset="DOC-OSHW-LOGO-" device="M" value="OSHW"/>
 <part name="J4" library="SPCoast" deviceset="CONNECTOR-RJ25" device="-6P6C" value="RJ12/6"/>
 <part name="X1" library="SPCoast" deviceset="KK-156-6" device="" value="0.156"/>
